File: cpe 2303l/cpe 2303l.kicad_sch (KiCad schematic)
At the start: 0 parts

Commit message: Add PCB and schematic files for project cpe 2303l
- Added a new backup ZIP file containing the PCB design and related files.
- Created a new KiCad project settings file (cpe 2303l.kicad_prl) with board configuration and visibility settings.
- Introduced an autosave lock file to manage concurrent editing sessions.
Parts:
- added BT1: Battery_Cell, Battery:BatteryHolder_Keystone_500, symbol Device:Battery_Cell
- added D1: LED, LED_THT:LED_D3.0mm_IRBlack, symbol Device:LED
- added R1: 100, Resistor_THT:R_Axial_DIN0204_L3.6mm_D1.6mm_P1.90mm_Vertical, symbol Device:R
Connections:
- new net: BT1.2 (-), D1.1 (K)
- new net: D1.2 (A), R1.2
- new net: BT1.1 (+), R1.1
