File: SEVILLA_PA1-2/SEVILLA_PA1-2.kicad_pcb (KiCad board)
At the start: 2 copper layers, 40 x 39 mm, 8 parts, among them SW1 SW_DIP_x02, U1 74LS04, U2 74LS08, U3 74LS32

Commit message: Add initial fp-info-cache file and include kicad-freerouting zip archive
Parts:
- moved R2 35.9 mm to (192.0, 125.0)
- moved R3 35.9 mm to (192.0, 128.1)
- moved D1 35.9 mm to (174.9, 122.0)
- moved R1 35.9 mm to (192.0, 121.8)
- moved SW1 35.9 mm to (181.1, 123.5)
- moved U2 35.9 mm to (185.5, 103.0)
- moved U3 35.9 mm to (196.3, 103.0)
- moved U1 35.9 mm to (174.7, 103.0)
Routing:
- net GND: track 0.00 -> 72.4 mm
- net Net-(R2-Pad1): track 0.00 -> 52.5 mm
- net Net-(R1-Pad1): track 0.00 -> 42.3 mm
- net Net-(D1-A): track 0.00 -> 38.7 mm
- net +5V: track 0.00 -> 23.5 mm
- net Net-(D1-K): track 0.00 -> 19.7 mm
- net Net-(U2-Pad6): track 0.00 -> 15.6 mm
- net Net-(U2-Pad3): track 0.00 -> 12.9 mm
- net Net-(U1-Pad2): track 0.00 -> 12.8 mm
- net Net-(U1-Pad4): track 0.00 -> 11.8 mm
- net Net-(SW1-Pad3): track 0.00 -> 2.54 mm
Other:
- board size 40 x 39 mm -> 42.5 x 36.5 mm
- board text added: "5V VCC"
- board text added: "74LS04"
- board text added: "74LS08"
- board text added: "74LS32"
- board text added: "CpE 2303L-2025-002 Rev 1.1"
- board text added: "GND"

Commit message: Refactor code structure for improved readability and maintainability
Other:
- board text added: "100"
- board text added: "5V"
- board text removed: "5V VCC"
Changed lines of the file:
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@@
+		)
+	)
+	(gr_text "100"
+		(at 201.5 128.5 0)
+		(layer "F.SilkS")
+		(effects
+			(font
+				(size 1 1)
+				(thickness 0.1)
+			)
+			(justify left bottom)
 		)
 	)
@@
 		)
 	)
-	(gr_text "5V VCC"
+	(gr_text "5V"
 		(at 205 103.5 0)
 		(layer "F.SilkS")
@@
 		)
 	)
-	(gr_text "5V VCC"
-		(at 192.5 100.5 0)
-		(layer "F.SilkS")
-		(effects
-			(font
-				(size 1 1)
-				(thickness 0.1)
-			)
-			(justify left bottom)
-		)
-	)
-	(gr_text "5V VCC"
-		(at 181.5 100.5 0)
+	(gr_text "5V"
+		(at 192.5 101.5 0)
+		(layer "F.SilkS")
+		(effects
+			(font
+				(size 1 1)
+				(thickness 0.1)
+			)
+			(justify left bottom)
+		)
+	)
+	(gr_text "100"
+		(at 201.5 122.5 0)
+		(layer "F.SilkS")
+		(effects
+			(font
+				(size 1 1)
+				(thickness 0.1)
+			)
+			(justify left bottom)
+		)
+	)
+	(gr_text "5V"
+		(at 181.18 101.645 0)
 		(layer "F.SilkS")
 		(effects
@@
 		)
 	)
+	(gr_text "100"
+		(at 201.5 125.5 0)
+		(layer "F.SilkS")
+		(effects
+			(font
+				(size 1 1)
+				(thickness 0.1)
+			)
+			(justify left bottom)
+		)
+	)
 	(gr_text "74LS08"
 		(at 187 100 0)
@@
 	)
 	(segment
-		(start 185.294 121.551)
-		(end 185 121.845)
+		(start 182.73 121.845)
+		(end 185.706 121.845)
 		(width 0.2)
 		(layer "B.Cu")
@@
 	)
 	(segment
-		(start 186 121.551)
-		(end 186.603 120.948)
-		(width 0.2)
-		(layer "B.Cu")
-		(net 3)
-	)
-	(segment
 		(start 185.8193 109.325)
 		(end 186.6045 110.1102)
@@
 	)
 	(segment
+		(start 181.085 123.49)
+		(end 182.73 121.845)
+		(width 0.2)
+		(layer "B.Cu")
+		(net 3)
+	)
+	(segment
 		(start 186.6045 113.6295)
 		(end 185.7679 114.4661)
@@
 	)
 	(segment
-		(start 182.73 121.845)
-		(end 181.085 123.49)
-		(width 0.2)
-		(layer "B.Cu")
-		(net 3)
-	)
-	(segment
-		(start 185 121.845)
-		(end 182.73 121.845)
-		(width 0.2)
-		(layer "B.Cu")
-		(net 3)
-	)
-	(segment
-		(start 186 121.551)
-		(end 185.294 121.551)
+		(start 185.706 121.845)
+		(end 186.603 120.948)
 		(width 0.2)
 		(layer "B.Cu")
@@
 	)
 	(segment
+		(start 179.9376 118)
+		(end 179.9376 118.215)
+		(width 0.2)
+		(layer "B.Cu")
+		(net 4)
+	)
+	(segment
 		(start 180.5 117.1037)
 		(end 184.3887 117.1037)
@@
 	(segment
 		(start 179.9376 117.6661)
-		(end 179.9376 118.215)
+		(end 179.9376 118)
 		(width 0.2)
 		(layer "B.Cu")
@@
 	)
 	(segment
+		(start 179.7226 118.215)
+		(end 179.9376 118)
+		(width 0.2)
+		(layer "B.Cu")
+		(net 4)
+	)
+	(segment
+		(start 174.72 118.215)
+		(end 179.7226 118.215)
+		(width 0.2)
+		(layer "B.Cu")
+		(net 4)
+	)
+	(segment
 		(start 180.2638 124.5955)
 		(end 186.0415 124.5955)
@@
 		(width 0.2)
 		(layer "B.Cu")
-		(net 4)
-	)
-	(segment
-		(start 174.72 118.215)
-		(end 179.9376 118.215)
-		(width 0.2)
-		(layer "B.Cu")

Commit message: Refactor code structure and remove redundant sections for improved readability and maintainability
Parts:
- moved R2 50.3 mm to (142.2, 118.3)
- moved U1 50.2 mm to (124.9, 97.3)
- moved U2 50.2 mm to (135.7, 97.3)
- moved U3 50.2 mm to (146.4, 97.3)
- moved R1 49.9 mm to (142.2, 122.3)
- moved SW1 43.3 mm to (137.8, 122.4), turned to 180 degrees
- moved R3 37.4 mm to (159.2, 110.3), turned to -90 degrees
- moved D1 22.6 mm to (159.4, 105.5), turned to 180 degrees
Routing:
- net Net-(D1-A): track 38.7 -> 11.8 mm
- net Net-(R2-Pad1): track 52.5 -> 67.5 mm
- net Net-(D1-K): track 19.7 -> 4.85 mm
- net GND: track 72.5 -> 63.0 mm
- net Net-(U1-Pad2): track 12.8 -> 11.8 mm
- net Net-(R1-Pad1): track 42.3 -> 43.0 mm
Other:
- board size 42.5 x 36.5 mm -> 40 x 34.5 mm
- board text added: "+"
- board text added: "-"
- board text added: "A"
- board text added: "B"

Commit message: Refactor code structure for improved readability and maintainability
Other:
- board size 40 x 34.5 mm -> 70 x 40 mm
- board text removed: "100"
Changed lines of the file:
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@@
 	)
 	(gr_rect
-		(start 122.66 92.825)
-		(end 162.66 127.325)
+		(start 108 90)
+		(end 178 130)
 		(stroke
 			(width 0.05)
@@
 	(gr_text "GND"
 		(at 147.6 112.825 0)
-		(layer "F.SilkS")
-		(effects
-			(font
-				(size 1 1)
-				(thickness 0.1)
-			)
-			(justify left bottom)
-		)
-	)
-	(gr_text "100"
-		(at 157.66 114.325 90)
 		(layer "F.SilkS")
 		(effects
@@
 		)
 	)
-	(gr_text "100"
-		(at 148.66 119.325 0)
-		(layer "F.SilkS")
-		(effects
-			(font
-				(size 1 1)
-				(thickness 0.1)
-			)
-			(justify left bottom)
-		)
-	)
 	(gr_text "5V"
 		(at 131.34 95.97 0)
@@
 	)
 	(gr_text "CpE 2303L-2025-002 Rev 1.1"
-		(at 136.66 126.825 0)
+		(at 153.5 129 0)
 		(layer "F.SilkS")
 		(effects
@@
 	(gr_text "+"
 		(at 156.16 107.825 0)
-		(layer "F.SilkS")
-		(effects
-			(font
-				(size 1 1)
-				(thickness 0.1)
-			)
-			(justify left bottom)
-		)
-	)
-	(gr_text "100"
-		(at 148.66 123.325 0)
 		(layer "F.SilkS")
 		(effects
@@
 		(layer "F.SilkS")
 		(effects
+			(font
+				(size 1 1)
+				(thickness 0.1)
+			)
+			(justify left bottom)
+		)
+	)
+	(gr_text "5V"
+		(at 126.5 120.5 0)
+		(layer "F.SilkS")
+		(effects
