File: SEVILLA_PA3-1/Power Supply.kicad_sch (KiCad schematic)
At the start: 11 parts, among them J10 5V OUTPUT, J7 Barrel_Jack_Switch, J8 11.1 V OUTPUT, J9 5V OUTPUT, U3 LM7809_TO220, U4 LM7805_TO220

Commit message: Refactor code structure and remove redundant sections for improved readability and maintainability
Connections:
- net GND: now also J7.2, J7.3
Other:
- title: Practical Activity #3 -> Practical Activity #3 Activity #1
Changed lines of the file:
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@@
 	(paper "USLetter")
 	(title_block
-		(title "Practical Activity #3")
+		(title "Practical Activity #3 Activity #1")
 		(date "2025-07-01")
 		(rev "1.0")
@@
 	)
 	(junction
+		(at 83.82 90.17)
+		(diameter 0)
+		(color 0 0 0 0)
+	)
+	(junction
 		(at 133.35 105.41)
 		(diameter 0)
@@
 	)
 	(junction
+		(at 90.17 105.41)
+		(diameter 0)
+		(color 0 0 0 0)
+	)
+	(junction
 		(at 175.26 96.52)
 		(diameter 0)
@@
 	(wire
 		(pts
+			(xy 83.82 90.17) (xy 83.82 105.41)
+		)
+		(stroke
+			(width 0)
+			(type default)
+		)
+	)
+	(wire
+		(pts
 			(xy 175.26 85.09) (xy 181.61 85.09)
 		)
@@
 		)
 		(stroke
+			(width 0)
+			(type default)
+		)
+	)
+	(wire
+		(pts
+			(xy 83.82 105.41) (xy 90.17 105.41)
+		)
+		(stroke
