File: SEVILLA_PA3-1/SEVILLA_PA3-1.kicad_sch (KiCad schematic)
At the start: 0 parts

Commit message: Refactor code structure and remove redundant sections for improved readability and maintainability
Other:
- title: Practical Activity #3 -> Practical Activity #3 Activity #1
Changed lines of the file:
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@@
 	(paper "USLetter")
 	(title_block
-		(title "Practical Activity #3")
+		(title "Practical Activity #3 Activity #1")
 		(date "2025-07-01")
 		(rev "1.0")
