File: SEVILLA_PA3-1/SEVILLA_PA3-1.kicad_pcb (KiCad board)
At the start: 2 copper layers, 66.8 x 58 mm, 19 parts, among them J1 MOTOR1 SIGNAL, J10 5V OUTPUT, J2 MOTOR1, J3 MOTOR2 SIGNAL, J4 MOTOR2, J5 MOTOR3 SIGNAL, J6 MOTOR3, J7 Barrel_Jack_Switch, J8 11.1 V OUTPUT, J9 5V OUTPUT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

Commit message: Add lock file for PCB design with hostname and username information
Other:
- board text added: "CpE 2303L-2024-004 Rev 1.0"
- board text removed: "CpE 2303L-2024-2025 Rev 1.0"
Changed lines of the file:
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@@
 		)
 	)
-	(gr_text "CpE 2303L-2024-2025 Rev 1.0"
+	(gr_text "CpE 2303L-2024-004 Rev 1.0"
 		(at 161.25 128.75 0)
 		(layer "B.SilkS")

Commit message: Refactor code structure and remove redundant sections for improved readability and maintainability
Parts:
- moved U1 18.5 mm to (121.4, 94.0), turned to 180 degrees
- moved U2 17.2 mm to (153.6, 93.7), turned to 180 degrees
- moved J6 13.5 mm to (160.8, 79.0), turned to 0 degrees
- moved J1 6.31 mm to (102.0, 80.2), turned to 0 degrees
- moved J4 6.27 mm to (107.0, 94.5), turned to 180 degrees
- moved J3 5.57 mm to (101.8, 92.5), turned to 0 degrees
- moved J5 4.95 mm to (161.0, 87.5), turned to 0 degrees
- moved J2 1.60 mm to (107.0, 79.8), turned to 0 degrees
Connections:
- J7 pad 2: Net-(J7-Pad2) -> GND
- J7 pad 3: Net-(J7-Pad2) -> GND
Routing:
- net /Motor Driver/FDIRECTION2: track 37.1 -> 0.00 mm
- net /Motor Driver/11.1V: track 157.1 -> 124.8 mm
- net /Motor Driver/BDIRECTION3: track 26.6 -> 0.00 mm
- net /Motor Driver/PWM2: track 19.5 -> 0.00 mm
- net /Motor Driver/BDIRECTION2: track 19.5 -> 0.00 mm
- net /Motor Driver/MOTOR3A: track 16.5 -> 0.00 mm
- net /Motor Driver/MOTOR1B: track 16.0 -> 0.00 mm
- net /Motor Driver/FDIRECTION1: track 15.8 -> 0.00 mm
- net /Motor Driver/MOTOR2A: track 15.7 -> 0.00 mm
- net /Motor Driver/MOTOR2B: track 14.3 -> 0.00 mm
- net /Motor Driver/BDIRECTION1: track 14.3 -> 0.00 mm
- net /Motor Driver/MOTOR3B: track 14.1 -> 0.00 mm
- net /Motor Driver/PWM3: track 14.1 -> 0.00 mm
- net /Motor Driver/FDIRECTION3: track 14.1 -> 0.00 mm
- net /Motor Driver/PWM1: track 13.6 -> 0.00 mm
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
Commit message: Refactor code structure and remove redundant sections for improved readability and maintainability
Parts:
- moved J1 30.3 mm to (132.0, 75.8), turned to 90 degrees
- moved J2 17.2 mm to (123.8, 75.7), turned to 90 degrees
- moved J3 16.3 mm to (102.5, 76.2)
- moved J7 6.25 mm to (114.5, 119.5)
- moved J4 5.17 mm to (102.5, 92.0)
- moved U1 2.32 mm to (119.1, 93.9)
Connections:
- net Net-(D1-A) renamed /Power Supply/LED
- net Net-(U3-VO) renamed /Power Supply/7809 Output
Routing:
- net /Motor Driver/FDIRECTION2: track 0.00 -> 26.4 mm
- net /Motor Driver/PWM1: track 0.00 -> 25.6 mm
- net /Motor Driver/FDIRECTION1: track 0.00 -> 22.0 mm
- net /Motor Driver/BDIRECTION3: track 0.00 -> 20.8 mm
- net /Motor Driver/MOTOR1A: track 0.00 -> 16.1 mm
- net /Motor Driver/BDIRECTION1: track 0.00 -> 15.5 mm
- net /Power Supply/7809 Output: track 0.00 -> 14.3 mm
- net /Motor Driver/MOTOR2B: track 0.00 -> 12.4 mm
- net /Motor Driver/MOTOR2A: track 0.00 -> 10.3 mm
- net /Motor Driver/MOTOR3A: track 0.00 -> 10.1 mm
- net /Motor Driver/BDIRECTION2: track 0.00 -> 10.0 mm
- net /Motor Driver/PWM2: track 0.00 -> 8.98 mm
- net /Motor Driver/11.1V: track 124.8 -> 133.5 mm
- net /Motor Driver/MOTOR3B: track 0.00 -> 8.00 mm
- net /Motor Driver/FDIRECTION3: track 0.00 -> 7.88 mm
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Other:
- board size 66.8 x 58 mm -> 66.8 x 60 mm
- board text added: "CpE 2303L-2024-004 Rev 1.1"
- board text removed: "CpE 2303L-2024-004 Rev 1.0"
