File: SEVILLA_PA4-2/SEVILLA_PA4-2.kicad_sch (KiCad schematic)
At the start: 15 parts, among them J1 Conn_01x02, SW3 SW_SPST, SW4 SW_SPST, U1 HDSP-7401, U2 PIC16F84A-XXP, U3 HDSP-7401, Y1 4 MHz

Commit message: Add lock files for PCB and schematic with user session details
- Created lock file for SEVILLA_PA4-2.kicad_pcb with hostname and username.
- Created lock file for SEVILLA_PA4-2.kicad_sch with hostname and username.
Connections:
- net GND: now also H1.1, H2.1, H3.1, H4.1
- no-connect marks 9 -> 5
Changed lines of the file:
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@@
+	)
+	(junction
+		(at 93.98 43.18)
+		(diameter 0)
+		(color 0 0 0 0)
 	)
 	(junction
@@
 	)
 	(junction
+		(at 115.57 43.18)
+		(diameter 0)
+		(color 0 0 0 0)
+	)
+	(junction
 		(at 176.53 105.41)
 		(diameter 0)
@@
 	)
 	(no_connect
-		(at 129.54 43.18)
-	)
-	(no_connect
-		(at 93.98 43.18)
-	)
-	(no_connect
 		(at 186.69 76.2)
-	)
-	(no_connect
-		(at 115.57 43.18)
-	)
-	(no_connect
-		(at 71.12 43.18)
 	)
 	(no_connect
@@
 	(wire
 		(pts
+			(xy 93.98 43.18) (xy 93.98 46.99)
+		)
+		(stroke
+			(width 0)
+			(type default)
+		)
+	)
+	(wire
+		(pts
 			(xy 168.91 109.22) (xy 177.8 109.22)
 		)
@@
 	(wire
 		(pts
+			(xy 115.57 43.18) (xy 129.54 43.18)
+		)
+		(stroke
+			(width 0)
+			(type default)
+		)
+	)
+	(wire
+		(pts
 			(xy 92.71 105.41) (xy 92.71 109.22)
 		)
@@
 	(wire
 		(pts
+			(xy 71.12 43.18) (xy 93.98 43.18)
+		)
+		(stroke
+			(width 0)
+			(type default)
+		)
+	)
+	(wire
+		(pts
 			(xy 177.8 102.87) (xy 186.69 102.87)
 		)
@@
 	(wire
 		(pts
+			(xy 93.98 43.18) (xy 115.57 43.18)
+		)
+		(stroke
+			(width 0)
+			(type default)
+		)
+	)
+	(wire
+		(pts
 			(xy 116.84 67.31) (xy 132.08 67.31)
 		)
@@
 		(pts
 			(xy 176.53 105.41) (xy 186.69 105.41)
+		)
+		(stroke
+			(width 0)
+			(type default)
+		)
+	)
+	(wire
+		(pts
+			(xy 93.98 46.99) (xy 102.87 46.99)
 		)
 		(stroke
@@
 				)
 				(justify left)
+				(hide yes)
 			)
 		)
@@
 	)
 	(symbol
+		(lib_id "power:GND")
+		(at 102.87 46.99 0)
+		(unit 1)
+		(exclude_from_sim no)
+		(in_bom yes)
+		(on_board yes)
+		(dnp no)
+		(fields_autoplaced yes)
+		(property "Reference" "#PWR08"
+			(at 102.87 53.34 0)
+			(effects
+				(font
+					(size 1.27 1.27)
+				)
+				(hide yes)
+			)
+		)
+		(property "Value" "GND"
+			(at 102.87 52.07 0)
+			(effects
+				(font
+					(size 1.27 1.27)
+				)
+			)
+		)
+		(property "Footprint" ""
+			(at 102.87 46.99 0)
+			(effects
+				(font
+					(size 1.27 1.27)
+				)
+				(hide yes)
+			)
+		)
+		(property "Datasheet" ""
+			(at 102.87 46.99 0)
+			(effects
+				(font
+					(size 1.27 1.27)
+				)
+				(hide yes)
+			)
+		)
+		(property "Description" "Power symbol creates a global label with name \"GND\" , ground"
+			(at 102.87 46.99 0)
+			(effects
+				(font
+					(size 1.27 1.27)
+				)
+				(hide yes)
+			)
+		)
+		(pin "1"
+		)
+		(instances
+			(project ""
+				(path "/65723761-f233-4867-895e-4aaa941e8e78"
+					(reference "#PWR08")
+					(unit 1)
+				)
+			)
+		)
+	)
+	(symbol
 		(lib_id "power:VCC")
 		(at 143.51 72.39 0)
@@
 				)
 				(justify left)
+				(hide yes)
 			)
 		)
@@
 				)
 				(justify left)
-			)
-		)
+				(hide yes)
+			)
+		)
