File: SEVILLA_PA5-2/SEVILLA_PA5-2.kicad_sch (KiCad schematic)
At the start: 11 parts, among them SW1 SW_DIP_x03, U1 74LS08, U2 74LS32, U3 74LS86

Commit message: Refactor code structure for improved readability and maintainability
Parts:
- removed SW1: SW_DIP_x03, symbol Switch:SW_DIP_x03
- added H1, H2, H3, H4: MountingHole_Pad, MountingHole:MountingHole_3.2mm_M3_DIN965_Pad, symbol Mechanical:MountingHole_Pad
- added SW2: ~, MyLibrary:MSG12ANG03, symbol MyLibrary:MSG12ANG03
- D2: footprint (none) -> LED_THT:LED_D3.0mm
Connections:
- net GND: now also H1.1, H2.1, H3.1, H4.1
- net at R3.1, U1.5, U3.5: now also SW2.3
- net VCC: now reaches R1.1, U1.1, U3.1
- net VCC: now also SW2.1
- net at R2.1, U1.2, U3.2: now also SW2.2
